Commit message: Model Update

File: catkin_ws/src/turtlebot3/turtlebot3_description/urdf/turtlebot3_burger.gazebo.xacro (robot description, xacro)
@@ -72,5 +72,5 @@
       <serviceName>imu_service</serviceName>
       <gaussianNoise>0.0</gaussianNoise>
-      <updateRate>200</updateRate>
+      <updateRate>10</updateRate>
       <imu>
         <noise>
@@ -101,12 +101,12 @@
         <scan>
           <horizontal>
-            <samples>360</samples>
+            <samples>10</samples>
             <resolution>1</resolution>
-            <min_angle>-1.5707975</min_angle>
-            <max_angle>1.5707975</max_angle>
+            <min_angle>-0.7854</min_angle>
+            <max_angle>0.7854</max_angle>
           </horizontal>
         </scan>
         <range>
-          <min>0.09</min>
+          <min>0.1</min>
           <max>3.5</max>
           <resolution>0.015</resolution>

File: catkin_ws/src/turtlebot3/turtlebot3_description/urdf/turtlebot3_burger.urdf.xacro (robot description, xacro)
@@ -170,15 +170,15 @@
   <gazebo reference="camera_link">
     <sensor type="camera" name="camera1">
-      <update_rate>30.0</update_rate>
+      <update_rate>10.0</update_rate>
       <camera name="head">
-        <horizontal_fov>1.3962634</horizontal_fov>
+        <horizontal_fov>1.085595</horizontal_fov>
         <image>
-          <width>304</width>
-          <height>228</height>
+          <width>640</width>
+          <height>192</height>
           <format>R8G8B8</format>
         </image>
         <clip>
-          <near>0.02</near>
-          <far>300</far>
+          <near>0.03</near>
+          <far>100</far>
         </clip>
         <noise>
@@ -193,5 +193,5 @@
       <plugin name="camera_controller" filename="libgazebo_ros_camera.so">
         <alwaysOn>true</alwaysOn>
-        <updateRate>0.0</updateRate>
+        <updateRate>10.0</updateRate>
         <cameraName>camera1</cameraName>
         <imageTopicName>image_raw</imageTopicName>
@@ -207,6 +207,6 @@
     </sensor>
   </gazebo>
-  <!-- bumper
-  <joint name="bumper_joint" type="fixed">
+  <!-- bumper -->
+  <!-- <joint name="bumper_joint" type="fixed">
     <axis xyz="0 1 0" />
     <origin xyz="0.05 0 0.02" rpy="0 0 0"/>
@@ -243,24 +243,7 @@
             </plugin>
             <always_on>true</always_on>
-            <update_rate>1000.</update_rate>
+            <update_rate>10</update_rate>
         </sensor>
     </gazebo>
-    -->
-    <!--
-    <gazebo reference="base_link">
-        <sensor name="collision_sensor" type="contact">
-            <plugin name="gazebo_ros_bumper_controller" filename="libgazebo_ros_bumper.so">
-                <bumpertopicname>bumper_vals</bumpertopicname>
-                <framename>world</framename>
-                <alwayson>true</alwayson>
-                <updaterate>1000.0</updaterate>
-            </plugin>
-            <always_on>true</always_on>
-            <update_rate>1000.</update_rate>
-            <contact>
-                <collision>base_footprint_fixed_joint_lump__bumper_collision_collision</collision>
-            </contact>
-        </sensor>
-    </gazebo>
-    -->
+     -->
 </robot>
